Commit message: update 25.12.23

File: src/haiheng-URDF/urdf/haiheng-URDF.urdf (robot description, URDF)
Before this commit: robot haiheng-URDF, 30 links, 29 joints
Joints:
- joint R_ELBOW_Y: limit lower=-1.37 upper=1.37 effort=9.6 velocity=3.87 -> lower=-1.36 upper=0.26 effort=9.6 velocity=3.87
- joint R_SHOULDER_P: limit lower=-3.1416 upper=3.1416 effort=30 velocity=3.56 -> lower=-1.49 upper=1.49 effort=30 velocity=3.56
- joint R_SHOULDER_R: limit lower=-1.19784 upper=1.49 effort=30 velocity=3.56 -> lower=-1.49 upper=1.49 effort=30 velocity=3.56
- joint R_SHOULDER_Y: limit lower=-3.1416 upper=3.1416 effort=9.6 velocity=3.87 -> lower=-2.36 upper=0.09 effort=9.6 velocity=3.87
- joint R_WRIST_P: limit lower=-3.1416 upper=4.70 effort=6.5 velocity=4.19 -> lower=0.79 upper=4.70 effort=6.5 velocity=4.19
- joint R_WRIST_R: limit lower=0 upper=1.94 effort=2.8 velocity=4.71 -> lower=0 upper=1.57 effort=2.8 velocity=4.71
